File: osu-keypad-4k/osu-keypad-4k.kicad_pcb (KiCad board)
At the start: 2 copper layers, 29 parts, among them SW1 SW_Push, U1 ATmega32U4-A, Y1 16MHz

Commit message: pcb
Parts:
- moved C5 40.5 mm to (191.8, 69.5), turned to 90 degrees
- moved C4 33.0 mm to (124.5, 71.1)
- moved Y1 32.4 mm to (186.7, 69.5), turned to 180 degrees
- moved R1 28.3 mm to (149.5, 74.0)
- moved R2 28.3 mm to (149.5, 71.4)
- moved C3 28.3 mm to (139.4, 72.4)
- moved C6 25.7 mm to (181.6, 69.5)
- moved USB1 9.16 mm to (162.6, 33.0), turned to 180 degrees
- moved C7 8.98 mm to (144.8, 68.6)
- moved D5 7.41 mm to (168.9, 47.0)
- moved R3 6.71 mm to (136.8, 64.8)
- moved U1 5.44 mm to (162.4, 65.1)
- moved C2 1.59 mm to (172.7, 54.3)
Routing:
- net GND: track 0.00 -> 68.8 mm
- net +5V: track 0.00 -> 27.4 mm
- net Net-(C6-Pad2): track 0.00 -> 16.7 mm
- net VCC: track 0.00 -> 7.68 mm
- net Net-(C5-Pad2): track 0.00 -> 4.02 mm
Other:
- board text added: "10uF"
